Commit message: update gr1t1 model

File: legged_examples/GR1T1/urdf/GR1T1.urdf (robot description, URDF)
Before this commit: robot GR1T1, 38 links, 37 joints
Links:
- removed link base
- removed link dummy_link
- added link base_link, mass 6.45116957899581; collision cylinder length=0.29 radius=0.039; visual mesh filename=package://gr1t1_description/meshes/base.STL
- added link imu_link
Joints:
- removed joint dummy_link_to_base
- added joint imu_joint: type fixed, parent base_link, child imu_link, origin xyz=0. 0. 0 rpy=0. 0. 0.
- joint l_hip_roll: parent base -> base_link
- joint r_hip_roll: parent base -> base_link
- joint waist_yaw: parent base -> base_link

Commit message: change toe and heel position

File: legged_examples/GR1T1/urdf/GR1T1.urdf (robot description, URDF)
Before this commit: robot GR1T1, 38 links, 37 joints
Joints:
- joint l_foot_heel_joint: origin xyz=-0.0445 0 -0.05 rpy=0 0 0 -> xyz=-0.07 0 -0.05 rpy=0 0 0
- joint l_foot_toe_joint: origin xyz=0.1415 0 -0.05 rpy=0 0 0 -> xyz=0.17 0 -0.05 rpy=0 0 0
- joint r_foot_heel_joint: origin xyz=-0.0445 0 -0.05 rpy=0 0 0 -> xyz=-0.07 0 -0.05 rpy=0 0 0
- joint r_foot_toe_joint: origin xyz=0.1415 0 -0.05 rpy=0 0 0 -> xyz=0.17 0 -0.05 rpy=0 0 0
