Commit message: update GR1T2 description; add h1 (6dof), high_torque

File: pybullet/assets/GR1T2/urdf/GR1T2_fixed_upper_body.urdf (robot description, URDF)
Before this commit: robot GR1T2, 39 links, 38 joints
Links:
- link base_link: geometry visual mesh filename=../meshes/base.STL
- link l_foot_pitch: geometry visual mesh filename=../meshes/Lleg5.STL
- link l_foot_roll: geometry collision cylinder length=0.24 radius=0.02; collision cylinder length=0.24 radius=0.02
- link l_hand_pitch: geometry collision sphere radius=0.036; visual mesh filename=../meshes/Larm7.STL
- link l_hand_roll: geometry visual mesh filename=../meshes/Larm6.STL
- link l_hand_yaw: geometry collision cylinder length=0.17 radius=0.035; visual mesh filename=../meshes/Larm5.STL
- link l_lower_arm_pitch: geometry visual mesh filename=../meshes/Larm4.STL
- link l_shank_pitch: geometry collision cylinder length=0.2 radius=0.05; visual mesh filename=../meshes/Lleg4.STL
- link l_thigh_pitch: geometry collision cylinder length=0.35 radius=0.05; visual mesh filename=../meshes/Lleg3.STL
- link l_thigh_roll: geometry visual mesh filename=../meshes/Lleg1.STL
- link l_thigh_yaw: geometry visual mesh filename=../meshes/Lleg2.STL
- link l_upper_arm_pitch: geometry visual mesh filename=../meshes/Larm1.STL
- link l_upper_arm_roll: geometry collision sphere radius=0.04; visual mesh filename=../meshes/Larm2.STL
- link l_upper_arm_yaw: geometry collision cylinder length=0.11 radius=0.03; visual mesh filename=../meshes/Larm3.STL
- link link_head_pitch: geometry collision sphere radius=0.07; visual mesh filename=../meshes/head3.STL
- link link_head_roll: geometry visual mesh filename=../meshes/head2.STL
- link link_head_yaw: geometry visual mesh filename=../meshes/head1.STL
- link link_waist_pitch: geometry visual mesh filename=../meshes/waist2.STL
- link link_waist_roll: geometry collision cylinder length=0.2 radius=0.1; visual mesh filename=../meshes/waist1.STL
- link link_waist_yaw: geometry visual mesh filename=../meshes/waist3.STL
- link r_foot_pitch: geometry visual mesh filename=../meshes/Rleg5.STL
- link r_foot_roll: geometry collision cylinder length=0.24 radius=0.02; collision cylinder length=0.24 radius=0.02
- link r_hand_pitch: geometry collision sphere radius=0.036; visual mesh filename=../meshes/Rarm7.STL
- link r_hand_roll: geometry visual mesh filename=../meshes/Rarm6.STL
- link r_hand_yaw: geometry collision cylinder length=0.17 radius=0.035; visual mesh filename=../meshes/Rarm5.STL
- link r_lower_arm_pitch: geometry visual mesh filename=../meshes/Rarm4.STL
- link r_shank_pitch: geometry collision cylinder length=0.2 radius=0.05; visual mesh filename=../meshes/Rleg4.STL
- link r_thigh_pitch: geometry collision cylinder length=0.35 radius=0.05; visual mesh filename=../meshes/Rleg3.STL
- link r_thigh_roll: geometry visual mesh filename=../meshes/Rleg1.STL
- link r_thigh_yaw: geometry visual mesh filename=../meshes/Rleg2.STL
- link r_upper_arm_pitch: geometry visual mesh filename=../meshes/Rarm1.STL
- link r_upper_arm_roll: geometry collision sphere radius=0.04; visual mesh filename=../meshes/Rarm2.STL
- link r_upper_arm_yaw: geometry collision cylinder length=0.11 radius=0.03; visual mesh filename=../meshes/Rarm3.STL
Joints:
- joint joint_head_pitch: type revolute -> fixed
- joint joint_head_roll: type revolute -> fixed
- joint joint_head_yaw: type revolute -> fixed
- joint joint_waist_pitch: type revolute -> fixed
- joint joint_waist_roll: type revolute -> fixed
- joint joint_waist_yaw: type revolute -> fixed
- joint l_elbow_pitch: type revolute -> fixed
- joint l_shoulder_pitch: type revolute -> fixed
- joint l_shoulder_roll: type revolute -> fixed
- joint l_shoulder_yaw: type revolute -> fixed
- joint l_wrist_pitch: type revolute -> fixed
- joint l_wrist_roll: type revolute -> fixed
- joint l_wrist_yaw: type revolute -> fixed
- joint r_elbow_pitch: type revolute -> fixed
- joint r_shoulder_pitch: type revolute -> fixed
- joint r_shoulder_roll: type revolute -> fixed
- joint r_shoulder_yaw: type revolute -> fixed
- joint r_wrist_pitch: type revolute -> fixed
- joint r_wrist_roll: type revolute -> fixed
- joint r_wrist_yaw: type revolute -> fixed
