Commit message: update GR1T2; add 3dof contact

File: legged_examples/GR1T2/urdf/GR1T2_no_visual.urdf (robot description, URDF)
Before this commit: robot GR1T2, 43 links, 42 joints
Links:
- removed link l_foot_heel_1
- removed link l_foot_heel_2
- removed link l_foot_toe_1
- removed link l_foot_toe_2
- removed link r_foot_heel_1
- removed link r_foot_heel_2
- removed link r_foot_toe_1
- removed link r_foot_toe_2
- added link l_foot_heel, mass 0.01
- added link l_foot_toe, mass 0.01
- added link r_foot_heel, mass 0.01
- added link r_foot_toe, mass 0.01
- link base_link: geometry 
- link l_foot_pitch: geometry 
- link l_foot_roll: geometry 
- link l_hand_pitch: geometry 
- link l_hand_roll: geometry 
- link l_hand_yaw: geometry 
- link l_lower_arm_pitch: geometry 
- link l_shank_pitch: geometry 
- link l_thigh_pitch: geometry 
- link l_thigh_roll: geometry 
- link l_thigh_yaw: geometry 
- link l_upper_arm_pitch: geometry 
- link l_upper_arm_roll: geometry 
- link l_upper_arm_yaw: geometry 
- link link_head_pitch: geometry 
- link link_head_roll: geometry 
- link link_head_yaw: geometry 
- link link_waist_pitch: geometry 
- link link_waist_roll: geometry 
- link link_waist_yaw: geometry 
- link r_foot_pitch: geometry 
- link r_foot_roll: geometry 
- link r_hand_pitch: geometry 
- link r_hand_roll: geometry 
- link r_hand_yaw: geometry 
- link r_lower_arm_pitch: geometry 
- link r_shank_pitch: geometry 
- link r_thigh_pitch: geometry 
- link r_thigh_roll: geometry 
- link r_thigh_yaw: geometry 
- link r_upper_arm_pitch: geometry 
- link r_upper_arm_roll: geometry 
- link r_upper_arm_yaw: geometry 
Joints:
- removed joint l_foot_heel_joint_1
- removed joint l_foot_heel_joint_2
- removed joint l_foot_toe_joint_1
- removed joint l_foot_toe_joint_2
- removed joint r_foot_heel_joint_1
- removed joint r_foot_heel_joint_2
- removed joint r_foot_toe_joint_1
- removed joint r_foot_toe_joint_2
- added joint leg_l5_fixed_1: type fixed, parent l_foot_roll, child l_foot_toe, origin xyz=0.1 0 -0.0300 rpy=0 0 0
- added joint leg_l5_fixed_2: type fixed, parent l_foot_roll, child l_foot_heel, origin xyz=-0.04 0 -0.0300 rpy=0 0 0
- added joint leg_r5_fixed_1: type fixed, parent r_foot_roll, child r_foot_toe, origin xyz=0.1 0 -0.0300 rpy=0 0 0
- added joint leg_r5_fixed_2: type fixed, parent r_foot_roll, child r_foot_heel, origin xyz=-0.040 0 -0.0300 rpy=0 0 0
