Commit message: wbc: add zero contact force constaint for additional 3dof contact; IK in reference generation (useless); uncommited changes for standing

File: legged_examples/GR1T2/urdf/GR1T2.urdf (robot description, URDF)
Before this commit: robot GR1T2, 43 links, 42 joints
Joints:
- joint l_foot_heel_joint_1: origin xyz=-0.07 0.02 -0.05 rpy=0 0 0 -> xyz=-0.04 0.0 -0.05 rpy=0 0 0
- joint l_foot_heel_joint_2: origin xyz=-0.07 -0.02 -0.05 rpy=0 0 0 -> xyz=-0.07 -0.04 -0.05 rpy=0 0 0
- joint l_foot_toe_joint_1: origin xyz=0.17 0.02 -0.05 rpy=0 0 0 -> xyz=0.10 0.0 -0.05 rpy=0 0 0
- joint l_foot_toe_joint_2: origin xyz=0.17 -0.02 -0.05 rpy=0 0 0 -> xyz=0.0 -0.04 -0.05 rpy=0 0 0
- joint r_foot_heel_joint_1: origin xyz=-0.07 -0.02 -0.05 rpy=0 0 0 -> xyz=-0.04 -0.0 -0.05 rpy=0 0 0
- joint r_foot_toe_joint_1: origin xyz=0.17 -0.02 -0.05 rpy=0 0 0 -> xyz=0.10 -0.0 -0.05 rpy=0 0 0
- joint r_foot_toe_joint_2: origin xyz=0.17 0.02 -0.05 rpy=0 0 0 -> xyz=0.0 0.04 -0.05 rpy=0 0 0

Commit message: add no contact motion task in wbc; change 3 dof contact positions for stable standing in mpc;

File: legged_examples/GR1T2/urdf/GR1T2.urdf (robot description, URDF)
Before this commit: robot GR1T2, 43 links, 42 joints
Joints:
- joint l_foot_heel_joint_1: origin xyz=-0.04 0.0 -0.05 rpy=0 0 0 -> xyz=-0.07 0.0 -0.05 rpy=0 0 0
- joint l_foot_toe_joint_1: origin xyz=0.10 0.0 -0.05 rpy=0 0 0 -> xyz=0.1 0.04 -0.05 rpy=0 0 0
- joint l_foot_toe_joint_2: origin xyz=0.0 -0.04 -0.05 rpy=0 0 0 -> xyz=0.1 -0.04 -0.05 rpy=0 0 0
- joint r_foot_heel_joint_1: origin xyz=-0.04 -0.0 -0.05 rpy=0 0 0 -> xyz=-0.07 -0.0 -0.05 rpy=0 0 0
- joint r_foot_toe_joint_1: origin xyz=0.10 -0.0 -0.05 rpy=0 0 0 -> xyz=0.1 -0.04 -0.05 rpy=0 0 0
- joint r_foot_toe_joint_2: origin xyz=0.0 0.04 -0.05 rpy=0 0 0 -> xyz=0.1 0.04 -0.05 rpy=0 0 0

Commit message: change contact position

File: legged_examples/GR1T2/urdf/GR1T2.urdf (robot description, URDF)
Before this commit: robot GR1T2, 43 links, 42 joints
Joints:
- joint l_foot_heel_joint_1: origin xyz=-0.07 0.0 -0.05 rpy=0 0 0 -> xyz=-0.07 0.04 -0.05 rpy=0 0 0
- joint r_foot_heel_joint_1: origin xyz=-0.07 -0.0 -0.05 rpy=0 0 0 -> xyz=-0.07 -0.04 -0.05 rpy=0 0 0
- joint r_foot_heel_joint_2: origin xyz=-0.07 0.02 -0.05 rpy=0 0 0 -> xyz=-0.07 0.04 -0.05 rpy=0 0 0

Commit message: change contact position

File: legged_examples/GR1T2/urdf/GR1T2.urdf (robot description, URDF)
Before this commit: robot GR1T2, 43 links, 42 joints
Joints:
- joint l_foot_toe_joint_1: origin xyz=0.1 0.04 -0.05 rpy=0 0 0 -> xyz=0.07 0.04 -0.05 rpy=0 0 0
- joint l_foot_toe_joint_2: origin xyz=0.1 -0.04 -0.05 rpy=0 0 0 -> xyz=0.07 -0.04 -0.05 rpy=0 0 0
- joint r_foot_toe_joint_1: origin xyz=0.1 -0.04 -0.05 rpy=0 0 0 -> xyz=0.07 -0.04 -0.05 rpy=0 0 0
- joint r_foot_toe_joint_2: origin xyz=0.1 0.04 -0.05 rpy=0 0 0 -> xyz=0.07 0.04 -0.05 rpy=0 0 0
